File: ts52k.kicad_sch (KiCad schematic)
At the start: 128 parts, among them J1 HRO_TYPE-C-31-M-12, J2 RGB, J3 ISP, SW1 SW_SPST, SW2 RotaryEncoder_Switch, U1 ATMEGA32U4, U2 TPD4E1U06, Y1 CSTNE16

Commit message: change to QFN
Parts:
- added C7: 0.1u, Capacitor_SMD:C_0402_1005Metric, symbol Device:C_Small
- added D6: WS2812B, LED_SMD:LED_WS2812B_PLCC4_5.0x5.0mm_P3.2mm, symbol LED:WS2812B
Connections:
- net +5V: now also C7.2, D6.1 (VDD)
- net GND: now also C7.1, D6.3 (VSS)
- net RGB: now also U1.36 (PF7(ADC7/TDI)), D6.4 (DIN); no longer J2.2 (Pin_2), U1.41 (PF0(ADC0))
- new net RGB2: D6.2 (DOUT), J2.2 (Pin_2)
Changed lines of the file:
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@@
   (junction (at 172.72 100.33) (diameter 0) (color 0 0 0 0)
   )
+  (junction (at 92.71 127.635) (diameter 0) (color 0 0 0 0)
+  )
   (junction (at 217.17 120.65) (diameter 0) (color 0 0 0 0)
   )
@@
   (no_connect (at 105.41 82.55))
   (no_connect (at 105.41 100.33))
-  (no_connect (at 105.41 41.91))
+  (no_connect (at 105.41 29.21))
   (no_connect (at 105.41 39.37))
   (no_connect (at 105.41 36.83))
@@
     (stroke (width 0) (type default) (color 0 0 0 0))
   )
+  (wire (pts (xy 95.25 127.635) (xy 92.71 127.635))
+    (stroke (width 0) (type default) (color 0 0 0 0))
+  )
   (wire (pts (xy 208.28 161.29) (xy 217.17 161.29))
     (stroke (width 0) (type default) (color 0 0 0 0))
@@
     )
   )
-  (global_label "RGB" (shape input) (at 185.42 33.02 180) (fields_autoplaced)
+  (global_label "RGB2" (shape input) (at 185.42 33.02 180) (fields_autoplaced)
     (effects (font (size 1.27 1.27)) (justify right))
-    (property "Intersheet References" "${INTERSHEET_REFS}" (id 0) (at 179.2858 32.9406 0)
+    (property "Intersheet References" "${INTERSHEET_REFS}" (id 0) (at 178.0763 32.9406 0)
       (effects (font (size 1.27 1.27)) (justify right) hide)
     )
@@
     )
   )
+  (global_label "RGB2" (shape input) (at 100.33 135.255 0) (fields_autoplaced)
+    (effects (font (size 1.27 1.27)) (justify left))
+    (property "Intersheet References" "${INTERSHEET_REFS}" (id 0) (at 107.6737 135.3344 0)
+      (effects (font (size 1.27 1.27)) (justify left) hide)
+    )
+  )
   (global_label "rpg1" (shape input) (at 263.525 79.375 0) (fields_autoplaced)
     (effects (font (size 1.27 1.27)) (justify left))
@@
     )
   )
-  (global_label "RGB" (shape input) (at 105.41 29.21 0) (fields_autoplaced)
+  (global_label "RGB" (shape input) (at 85.09 135.255 180) (fields_autoplaced)
+    (effects (font (size 1.27 1.27)) (justify right))
+    (property "Intersheet References" "${INTERSHEET_REFS}" (id 0) (at 50.8 13.335 0)
+      (effects (font (size 1.27 1.27)) hide)
+    )
+  )
+  (global_label "RGB" (shape input) (at 105.41 41.91 0) (fields_autoplaced)
     (effects (font (size 1.27 1.27)) (justify left))
-    (property "Intersheet References" "${INTERSHEET_REFS}" (id 0) (at 0 -5.08 0)
+    (property "Intersheet References" "${INTERSHEET_REFS}" (id 0) (at 0 7.62 0)
       (effects (font (size 1.27 1.27)) hide)
     )
@@
     (pin "1")
   )
+  (symbol (lib_id "power:GND") (at 100.33 127.635 90) (unit 1)
+    (in_bom yes) (on_board yes)
+    (property "Reference" "#PWR04" (id 0) (at 106.68 127.635 0)
+      (effects (font (size 1.27 1.27)) hide)
+    )
+    (property "Value" "GND" (id 1) (at 103.5812 127.508 90)
+      (effects (font (size 1.27 1.27)) (justify right) hide)
+    )
+    (property "Footprint" "" (id 2) (at 100.33 127.635 0)
+      (effects (font (size 1.27 1.27)) hide)
+    )
+    (property "Datasheet" "" (id 3) (at 100.33 127.635 0)
+      (effects (font (size 1.27 1.27)) hide)
+    )
+    (pin "1")
+  )
+  (symbol (lib_id "power:GND") (at 92.71 142.875 0) (unit 1)
+    (in_bom yes) (on_board yes)
+    (property "Reference" "#PWR03" (id 0) (at 92.71 149.225 0)
+      (effects (font (size 1.27 1.27)) hide)
+    )
+    (property "Value" "GND" (id 1) (at 92.837 147.2692 0))
+    (property "Footprint" "" (id 2) (at 92.71 142.875 0)
+      (effects (font (size 1.27 1.27)) hide)
+    )
+    (property "Datasheet" "" (id 3) (at 92.71 142.875 0)
+      (effects (font (size 1.27 1.27)) hide)
+    )
+    (pin "1")
+  )
   (symbol (lib_id "power:GND") (at 267.335 71.12 90) (unit 1)
     (in_bom yes) (on_board yes)
@@
     (pin "2")
   )
+  (symbol (lib_id "LED:WS2812B") (at 92.71 135.255 0) (unit 1)
+    (in_bom yes) (on_board yes)
+    (property "Reference" "D6" (id 0) (at 95.25 142.875 0)
+      (effects (font (size 1.27 1.27)) (justify left))
+    )
+    (property "Value" "WS2812B" (id 1) (at 95.25 145.415 0)
+      (effects (font (size 1.27 1.27)) (justify left))
+    )
+    (property "Footprint" "LED_SMD:LED_WS2812B_PLCC4_5.0x5.0mm_P3.2mm" (id 2) (at 93.98 142.875 0)
+      (effects (font (size 1.27 1.27)) (justify left top) hide)
+    )
+    (property "Datasheet" "https://cdn-shop.adafruit.com/datasheets/WS2812B.pdf" (id 3) (at 95.25 144.78 0)
+      (effects (font (size 1.27 1.27)) (justify left top) hide)
+    )
+    (property "LCSC" "C114586" (id 4) (at 92.71 135.255 0)
+      (effects (font (size 1.27 1.27)) hide)
+    )
+    (pin "1")
+    (pin "2")
+    (pin "3")
+    (pin "4")
+  )
+  (symbol (lib_id "Device:C_Small") (at 97.79 127.635 270) (unit 1)
+    (in_bom yes) (on_board yes)
+    (property "Reference" "C7" (id 0) (at 97.79 121.8184 90))
+    (property "Value" "0.1u" (id 1) (at 97.79 124.1298 90))
+    (property "Footprint" "Capacitor_SMD:C_0402_1005Metric" (id 2) (at 97.79 127.635 0)
+      (effects (font (size 1.27 1.27)) hide)
+    )
+    (property "Datasheet" "~" (id 3) (at 97.79 127.635 0)
+      (effects (font (size 1.27 1.27)) hide)
+    )
+    (property "LCSC" "C60474" (id 4) (at 97.79 127.635 0)
+      (effects (font (size 1.27 1.27)) hide)
+    )
+    (pin "1")
+    (pin "2")
+  )
+  (symbol (lib_id "power:+5V") (at 92.71 127.635 0) (unit 1)
+    (in_bom yes) (on_board yes)
+    (property "Reference" "#PWR02" (id 0) (at 92.71 131.445 0)
+      (effects (font (size 1.27 1.27)) hide)
+    )
+    (property "Value" "+5V" (id 1) (at 93.091 123.2408 0))
+    (property "Footprint" "" (id 2) (at 92.71 127.635 0)
+      (effects (font (size 1.27 1.27)) hide)
+    )
+    (property "Datasheet" "" (id 3) (at 92.71 127.635 0)
+      (effects (font (size 1.27 1.27)) hide)
+    )
+    (pin "1")
+  )
   (symbol (lib_id "Device:C_Small") (at 260.985 67.945 180) (unit 1)
     (in_bom yes) (on_board yes)
@@
   )
   (symbol_instances
+    (path "/c52532d0-384f-437f-8337-e761429d3390"
+      (reference "#PWR02") (unit 1) (value "+5V") (footprint "")
+    )
+    (path "/1d796767-159a-4540-856b-1f2de524ef3b"
+      (reference "#PWR03") (unit 1) (value "GND") (footprint "")
+    )
+    (path "/0c11cd35-26cc-4a1c-a433-f9b838604d23"
+      (reference "#PWR04") (unit 1) (value "GND") (footprint "")
+    )
     (path "/00000000-0000-0000-0000-00006179a9d0"
       (reference "#PWR0101") (unit 1) (value "GND") (footprint "")
@@
       (reference "C6") (unit 1) (value "4.7u") (footprint "Capacitor_SMD:C_0603_1608Metric")
     )
+    (path "/7f9397e0-40de-4baa-89e1-1921167c4577"
+      (reference "C7") (unit 1) (value "0.1u") (footprint "Capacitor_SMD:C_0402_1005Metric")
+    )
     (path "/2a817ce4-6235-40a2-a6dd-46495631cc6c"
       (reference "C19") (unit 1) (value "0.1u") (footprint "Capacitor_SMD:C_0402_1005Metric")
@@
       (reference "D5") (unit 1) (value "D") (footprint "Diode_SMD:D_SOD-123")
     )
+    (path "/4d6768dc-b381-4c41-b8ba-d87395ee35ee"
+      (reference "D6") (unit 1) (value "WS2812B") (footprint "LED_SMD:LED_WS2812B_PLCC4_5.0x5.0mm_P3.2mm")
+    )
     (path "/00000000-0000-0000-0000-0000613c2aa2"

Commit message: jlcpcb ordered
Parts:
- added R7: Open, Resistor_SMD:R_0603_1608Metric, symbol Device:R_Small
- added R8: 330, Resistor_SMD:R_0603_1608Metric, symbol Device:R_Small
- C1: LCSC C5673 -> C15849
- C19, C2, C20, C3, C5, C7: LCSC C60474 -> C1525
- C4: footprint Capacitor_SMD:C_0402_1005Metric -> Capacitor_SMD:C_0603_1608Metric; LCSC C60474 -> C1525
- C6: LCSC C1705 -> C19666
- D11, D12, D13, D14, D16, D17, D18, D2, D20, D21, D22, D23, D25, D26, D27, D29, D3, D30, D31, D33, D34, D35, D37, D38, D39, D4, D40, D42, D43, D44, D46, D47, D48, D49, D5, D51, D52, D53, D55, D56, D58, D61, D63, D64, D65, D66, D68, D7, D70, D8, D87, D88, D9: LCSC C84367 -> C81598
- R1, R4: LCSC C269742 -> C17414
- R2, R3: LCSC C269708 -> C23345
- R5, R6: LCSC C269716 -> C23186
- SW1: LCSC C780528 -> C318884
- U1: LCSC C44854 -> C112161
Connections:
- net RGB: now also R8.1; no longer D6.4 (DIN)
- net RGB2: now also R7.1
- new net: D6.4 (DIN), R7.2, R8.2
